Commit message: no slider,jacobian and TF added

File: first_leg/scripts/leg_RBDL.urdf (robot description, URDF)
Before this commit: robot leg, 7 links, 6 joints
Links:
- removed link jump
- removed link world
- added link trunk_inertia
- link trunk: geometry collision box size=0.3 0.2 0.1; visual box size=0.3 0.2 0.1
Joints:
- removed joint jumper
- removed joint trunk_to_world
- added joint trunk_to_trunk_inertia: type fixed, parent trunk_inertia, child trunk, origin xyz=0 0 0 rpy=0 0 0
- joint hip_joint: origin xyz=0.02 0 0 rpy=0 0 0 -> xyz=0.15 0.07 0.05 rpy=0 0 0; parent jump -> trunk

File: first_leg/urdf/leg_no_slider.urdf (robot description, URDF)
Before this commit: robot leg, 7 links, 6 joints
Links:
- removed link jump
- link trunk: geometry collision box size=0.3 0.2 0.1; visual box size=0.3 0.2 0.1
Joints:
- removed joint jumper
- joint hip_joint: origin xyz=0.02 0 0 rpy=0 0 0 -> xyz=0.15 0.07 0.05 rpy=0 0 0; parent jump -> trunk

Commit message: frames are fixed

File: first_leg/scripts/leg_RBDL.urdf (robot description, URDF)
Before this commit: robot leg, 6 links, 5 joints
Links:
- link thigh: geometry collision box size=0.06 0.07125 0.2131; visual box size=0.06 0.07125 0.2131
Joints:
- joint calf_joint: origin xyz=0 0.01 -0.1881 rpy=0 0 0 -> xyz=0 0.07125 -0.2131 rpy=0 0 0
- joint foot_fixed: origin xyz=0 0.01 -0.1881 rpy=0 0 0 -> xyz=0 0 -0.21148 rpy=0 0 0
- joint hip_joint: origin xyz=0.15 0.07 0.05 rpy=0 0 0 -> xyz=0.15 0.07 0 rpy=0 0 0
- joint thigh_joint: origin xyz=0.03 0.04 0 rpy=0 0 0 -> xyz=0.06 0.015 0 rpy=0 0 0

File: first_leg/urdf/leg_no_slider.urdf (robot description, URDF)
Before this commit: robot leg, 6 links, 5 joints
Links:
- link thigh: geometry collision box size=0.06 0.07125 0.2131; visual box size=0.06 0.07125 0.2131
Joints:
- joint calf_joint: origin xyz=0 0.01 -0.2131 rpy=0 0 0 -> xyz=0 0.07125 -0.2131 rpy=0 0 0
- joint foot_fixed: origin xyz=0 0.01 -0.21148 rpy=0 0 0 -> xyz=0 0 -0.21148 rpy=0 0 0
- joint hip_joint: origin xyz=0.15 0.07 0.05 rpy=0 0 0 -> xyz=0.15 0.07 0 rpy=0 0 0
- joint thigh_joint: origin xyz=0.03 0.04 0 rpy=0 0 0 -> xyz=0.06 0.015 0 rpy=0 0 0

Commit message: urdf update

File: first_leg/scripts/leg_RBDL.urdf (robot description, URDF)
Before this commit: robot leg, 6 links, 5 joints
Links:
- link calf: geometry collision box size=0.03 0.02 0.240; visual box size=0.03 0.02 0.240
Joints:
- joint foot_fixed: origin xyz=0 0 -0.21148 rpy=0 0 0 -> xyz=0 0 -0.240 rpy=0 0 0

File: first_leg/urdf/leg_no_slider.urdf (robot description, URDF)
Before this commit: robot leg, 6 links, 5 joints
Links:
- link calf: geometry collision box size=0.03 0.02 0.240; visual box size=0.03 0.02 0.240
- link thigh: geometry collision box size=0.06 0.07125 0.21183; visual box size=0.06 0.07125 0.21183
Joints:
- joint calf_joint: origin xyz=0 0.07125 -0.2131 rpy=0 0 0 -> xyz=0 0.07125 -0.21183 rpy=0 0 0
- joint foot_fixed: origin xyz=0 0 -0.21148 rpy=0 0 0 -> xyz=0 0 -0.240 rpy=0 0 0

Commit message: urdf fixed - circule node added

File: first_leg/scripts/leg_RBDL.urdf (robot description, URDF)
Before this commit: robot leg, 6 links, 5 joints
Links:
- removed link trunk_inertia
- added link world
- link foot: mass 0.05 -> 0.005
- link thigh: geometry collision box size=0.06 0.07125 0.21183; visual box size=0.06 0.07125 0.21183
- link trunk: geometry collision box size=0.1 0.06 0.09; visual box size=0.1 0.06 0.09
Joints:
- removed joint trunk_to_trunk_inertia
- added joint trunk_to_world: type fixed, parent world, child trunk, origin xyz=0 0 0.0 rpy=0 0 0
- joint calf_joint: origin xyz=0 0.07125 -0.2131 rpy=0 0 0 -> xyz=0 0.07125 -0.21183 rpy=0 0 0
- joint hip_joint: limit lower=-0.872664625997 upper=1.0471975512 effort=20 velocity=1.6 -> lower=-3.14 upper=3.14 effort=20 velocity=1.6; origin xyz=0.03 0 0.9 rpy=0 0 0 -> xyz=0.05 0 0.0 rpy=0 0 0

File: first_leg/urdf/leg_no_slider.urdf (robot description, URDF)
Before this commit: robot leg, 6 links, 5 joints
Links:
- link trunk: geometry collision box size=0.1 0.06 0.09; visual box size=0.1 0.06 0.09
Joints:
- joint hip_joint: origin xyz=0.03 0 0.9 rpy=0 0 0 -> xyz=0.05 0 0.0 rpy=0 0 0
- joint trunk_to_world: origin xyz=0 0 0 rpy=0 0 0 -> xyz=0 0 0.0 rpy=0 0 0
