Commit message: urdf changed and pose node added

File: first_leg/scripts/legRBDL.urdf (robot description, URDF)
Before this commit: robot leg, 7 links, 6 joints
Links:
- removed link foot
- removed link jump
- removed link world
- added link trunk_inertia
- link calf: geometry collision box size=0.05 0.02 0.21148; visual box size=0.05 0.02 0.21148
- link trunk: mass 100 -> 3.3; geometry collision box size=0.3 0.2 1; visual box size=0.3 0.2 1
Joints:
- removed joint foot_fixed
- removed joint jumper
- removed joint trunk_to_world
- added joint trunk_to_trunk_inertia: type fixed, parent trunk_inertia, child trunk, origin xyz=0 0 0 rpy=0 0 0
- joint calf_joint: limit lower=-3.14159265359 upper=3.14159265359 effort=20 velocity=1.6 -> lower=-3.14159265359 upper=3.14159265359 effort=20 velocity=10.6; origin xyz=0 0.01 -0.1881 rpy=0 0 0 -> xyz=0 0 -0.2131 rpy=0 0 0
- joint hip_joint: limit lower=-0.872664625997 upper=1.0471975512 effort=20 velocity=1.6 -> lower=-0.872664625997 upper=1.0471975512 effort=20 velocity=10.6; origin xyz=0.02 0 0 rpy=0 0 0 -> xyz=0.15 0.06 0 rpy=0 0 0; parent jump -> trunk
- joint thigh_joint: limit lower=-0.523598775598 upper=3.92699081699 effort=20 velocity=1.6 -> lower=-0.523598775598 upper=3.92699081699 effort=20 velocity=10.6

Commit message: nodes and legRBDL updated

File: first_leg/scripts/legRBDL.urdf (robot description, URDF)
Before this commit: robot leg, 5 links, 4 joints
Links:
- added link jump, mass 0.002; collision box size=0.02 0.08 0.093; visual box size=0.02 0.08 0.093
Joints:
- added joint jumper: type prismatic, parent trunk, child jump, origin xyz=0.15 0.07 0.9 rpy=0 0 0, axis 0 0 1, limit lower=-0.2 upper=0.5 effort=20 velocity=0.5
- joint hip_joint: limit lower=-0.872664625997 upper=1.0471975512 effort=20 velocity=10.6 -> lower=-0.872664625997 upper=1.0471975512 effort=20 velocity=1.6; origin xyz=0.15 0.06 0 rpy=0 0 0 -> xyz=0.02 0 0 rpy=0 0 0; parent trunk -> jump

Commit message: legRBDL.urdf fixed command_slider added

File: first_leg/scripts/legRBDL.urdf (robot description, URDF)
Before this commit: robot leg, 6 links, 5 joints
Links:
- added link foot, mass 0.005; collision sphere radius=0.025; visual sphere radius=0.025
- link calf: geometry collision box size=0.03 0.02 0.21148; visual box size=0.03 0.02 0.21148
- link thigh: geometry collision box size=0.06 0.07125 0.2131; visual box size=0.06 0.07125 0.2131
- link trunk: mass 3.3 -> 100; geometry collision box size=0.06 0.06 1.5; visual box size=0.06 0.06 1.5
Joints:
- removed joint jumper
- added joint foot_fixed: type fixed, parent calf, child foot, origin xyz=0 0 -0.21148 rpy=0 0 0, axis 0 1 0, limit lower=-3.14159265359 upper=3.14159265359 effort=20 velocity=10.6
- joint calf_joint: limit lower=-3.14159265359 upper=3.14159265359 effort=20 velocity=10.6 -> lower=-3.14159265359 upper=3.14159265359 effort=20 velocity=1.6; origin xyz=0 0 -0.2131 rpy=0 0 0 -> xyz=0 0.07125 -0.2131 rpy=0 0 0
- joint hip_joint: origin xyz=0.02 0 0 rpy=0 0 0 -> xyz=0.03 0 0 rpy=0 0 0
- joint thigh_joint: limit lower=-0.523598775598 upper=3.92699081699 effort=20 velocity=10.6 -> lower=-0.523598775598 upper=3.92699081699 effort=20 velocity=1.6; origin xyz=0.03 0.04 0 rpy=0 0 0 -> xyz=0.06 0.015 0 rpy=0 0 0

File: first_leg/urdf/leg.urdf (robot description, URDF)
Before this commit: robot leg, 7 links, 6 joints
Links:
- link foot: mass 0.05 -> 0.005
- link thigh: geometry collision box size=0.06 0.07125 0.2131; visual box size=0.06 0.07125 0.2131
- link trunk: geometry collision box size=0.06 0.06 1.5; visual box size=0.06 0.06 1.5
Joints:
- joint calf_joint: origin xyz=0 0.01 -0.2131 rpy=0 0 0 -> xyz=0 0.07125 -0.2131 rpy=0 0 0
- joint foot_fixed: origin xyz=0 0.01 -0.21148 rpy=0 0 0 -> xyz=0 0 -0.21148 rpy=0 0 0
- joint hip_joint: origin xyz=0.02 0 0 rpy=0 0 0 -> xyz=0.03 0 0 rpy=0 0 0
- joint jumper: origin xyz=0.15 0.07 0.9 rpy=0 0 0 -> xyz=0 0 0.9 rpy=0 0 0
- joint thigh_joint: origin xyz=0.03 0.04 0 rpy=0 0 0 -> xyz=0.06 0.015 0 rpy=0 0 0

File: first_leg/urdf/leg_no_slider.urdf (robot description, URDF)
Before this commit: robot leg, 6 links, 5 joints
Links:
- link foot: mass 0.05 -> 0.005

Commit message: world coordinates are similar

File: first_leg/scripts/legRBDL.urdf (robot description, URDF)
Before this commit: robot leg, 7 links, 5 joints
Joints:
- added joint jumper: type prismatic, parent trunk, child jump, origin xyz=0 0 0.9 rpy=0 0 0, axis 0 0 1, limit lower=-0.2 upper=0.5 effort=20 velocity=0.5

File: first_leg/scripts/leg_RBDL.urdf (robot description, URDF)
Before this commit: robot leg, 6 links, 5 joints
Links:
- link trunk: geometry collision box size=0.06 0.06 1.5; visual box size=0.06 0.06 1.5
Joints:
- joint hip_joint: origin xyz=0.15 0.07 0 rpy=0 0 0 -> xyz=0.03 0 0.9 rpy=0 0 0

File: first_leg/urdf/leg_no_slider.urdf (robot description, URDF)
Before this commit: robot leg, 6 links, 5 joints
Links:
- link trunk: geometry collision box size=0.06 0.06 1.5; visual box size=0.06 0.06 1.5
Joints:
- joint hip_joint: origin xyz=0.15 0.07 0 rpy=0 0 0 -> xyz=0.03 0 0.9 rpy=0 0 0

Commit message: prismatic joint problem fixed

File: first_leg/scripts/legRBDL.urdf (robot description, URDF)
Before this commit: robot leg, 7 links, 6 joints
Joints:
- joint jumper: limit lower=-0.2 upper=0.5 effort=20 velocity=0.5 -> lower=-0.7 upper=0.5 effort=20 velocity=0.5

File: first_leg/urdf/leg.urdf (robot description, URDF)
Before this commit: robot leg, 7 links, 6 joints
Joints:
- joint jumper: limit lower=-0.2 upper=0.5 effort=20 velocity=0.5 -> lower=-0.7 upper=0.5 effort=20 velocity=0.5

Commit message: urdf for slider/pose slider added in robot class

File: first_leg/scripts/legRBDL.urdf (robot description, URDF)
Before this commit: robot leg, 7 links, 6 joints
Links:
- link calf: geometry collision box size=0.03 0.02 0.240; visual box size=0.03 0.02 0.240
- link thigh: geometry collision box size=0.06 0.07125 0.21183; visual box size=0.06 0.07125 0.21183
Joints:
- joint calf_joint: origin xyz=0 0.07125 -0.2131 rpy=0 0 0 -> xyz=0 0.07125 -0.21183 rpy=0 0 0
- joint foot_fixed: origin xyz=0 0 -0.21148 rpy=0 0 0 -> xyz=0 0 -0.240 rpy=0 0 0
- joint hip_joint: origin xyz=0.03 0 0 rpy=0 0 0 -> xyz=0.05 0 0 rpy=0 0 0

File: first_leg/urdf/leg.urdf (robot description, URDF)
Before this commit: robot leg, 7 links, 6 joints
Links:
- link calf: geometry collision box size=0.03 0.02 0.240; visual box size=0.03 0.02 0.240
- link thigh: geometry collision box size=0.06 0.07125 0.21183; visual box size=0.06 0.07125 0.21183
Joints:
- joint calf_joint: origin xyz=0 0.07125 -0.2131 rpy=0 0 0 -> xyz=0 0.07125 -0.21183 rpy=0 0 0
- joint foot_fixed: origin xyz=0 0 -0.21148 rpy=0 0 0 -> xyz=0 0 -0.240 rpy=0 0 0
- joint hip_joint: origin xyz=0.03 0 0 rpy=0 0 0 -> xyz=0.05 0 0 rpy=0 0 0

Commit message: mass eddited and ground force added

File: first_leg/scripts/legRBDL.urdf (robot description, URDF)
Before this commit: robot leg, 7 links, 6 joints
Links:
- link calf: mass 0.133 -> 0.204
- link hip: mass 0.63 -> 0.654
- link thigh: mass 1.062 -> 1.154

File: first_leg/urdf/leg.urdf (robot description, URDF)
Before this commit: robot leg, 7 links, 6 joints
Links:
- link calf: mass 0.133 -> 0.204
- link hip: mass 0.63 -> 0.654
- link thigh: mass 1.062 -> 1.154
Joints:
- joint jumper: limit lower=-0.7 upper=0.5 effort=20 velocity=0.5 -> lower=-0.7 upper=0.5 effort=10000 velocity=0.5

Commit message: hopper model in gazebo

File: first_leg/scripts/legRBDL.urdf (robot description, URDF)
Before this commit: robot leg, 7 links, 6 joints
Links:
- link calf: mass 0.204 -> 0.133
- link hip: mass 0.654 -> 0.63
- link thigh: mass 1.154 -> 1.062

File: first_leg/urdf/hardware.urdf (robot description, URDF)
Before this commit: robot leg, 7 links, 6 joints
Links:
- removed link jump
- link trunk: geometry collision box size=0.1 0.06 0.09; visual box size=0.1 0.06 0.09
Joints:
- removed joint jumper
- joint calf_joint: limit lower=-3.14159265359 upper=0.0 effort=1000 velocity=100 -> lower=-3.14159265359 upper=3.14159265359 effort=20 velocity=1.6
- joint foot_fixed: limit lower=0 upper=0 effort=1 velocity=1 -> lower=-3.14159265359 upper=3.14159265359 effort=20 velocity=10.6; type revolute -> fixed
- joint hip_joint: limit lower=-0.872664625997 upper=1.0471975512 effort=10 velocity=5 -> lower=-3.14 upper=3.14 effort=20 velocity=1.6; parent jump -> trunk
- joint thigh_joint: limit lower=-0.523598775598 upper=3.92699081699 effort=10 velocity=5 -> lower=-0.523598775598 upper=3.92699081699 effort=20 velocity=1.6

File: first_leg/urdf/leg_no_slider.urdf (robot description, URDF)
Before this commit: robot leg, 6 links, 5 joints
Links:
- link trunk: mass 100 -> 0.001

Commit message: slip model edit

File: first_leg/scripts/legRBDL.urdf (robot description, URDF)
Before this commit: robot leg, 7 links, 6 joints
Links:
- link jump: mass 0.002 -> 2.18

File: first_leg/urdf/leg.urdf (robot description, URDF)
Before this commit: robot leg, 7 links, 6 joints
Joints:
- joint jumper: origin xyz=0 0 0.5 rpy=0 0 0 -> xyz=0 0 0.9 rpy=0 0 0
