Commit message: cammand node added and urdf is fixed now

File: first_leg/urdf/leg.urdf (robot description, URDF)
Before this commit: robot leg, 7 links, 6 joints
Joints:
- joint calf_joint: origin xyz=0 0.01 -0.1881 rpy=0 0 0 -> xyz=0 0.01 -0.2131 rpy=0 0 0
- joint foot_fixed: origin xyz=0 0.01 -0.1881 rpy=0 0 0 -> xyz=0 0.01 -0.21148 rpy=0 0 0

File: first_leg/urdf/leg_no_slider.urdf (robot description, URDF)
Before this commit: robot leg, 6 links, 5 joints
Joints:
- joint calf_joint: origin xyz=0 0.01 -0.1881 rpy=0 0 0 -> xyz=0 0.01 -0.2131 rpy=0 0 0
- joint foot_fixed: origin xyz=0 0.01 -0.1881 rpy=0 0 0 -> xyz=0 0.01 -0.21148 rpy=0 0 0

Commit message: calculate lambda in robot class

File: first_leg/urdf/leg.urdf (robot description, URDF)
Before this commit: robot leg, 7 links, 6 joints
Joints:
- joint calf_joint: limit lower=-3.14159265359 upper=3.14159265359 effort=20 velocity=1.6 -> lower=-3.14159265359 upper=0.0 effort=20 velocity=1.6

Commit message: test_jump and robot_class eddited

File: first_leg/urdf/leg.urdf (robot description, URDF)
Before this commit: robot leg, 7 links, 6 joints
Links:
- link jump: mass 0.002 -> 2.18
- link thigh: geometry collision box size=0.03 0.02 0.1; visual box size=0.06 0.07125 0.21183
Joints:
- removed joint foot_fixed
- added joint foot_joint: type revolute, parent calf, child foot, origin xyz=0 0 -0.240 rpy=0 0 0, axis 0 1 0, limit lower=0 upper=0 effort=1 velocity=1
- joint hip_joint: limit lower=-0.872664625997 upper=1.0471975512 effort=10 velocity=5 -> lower=-0.872664625997 upper=1.0471975512 effort=100 velocity=5
- joint jumper: limit lower=-0.7 upper=0.5 effort=1000 velocity=50 -> lower=-1 upper=0.5 effort=1000 velocity=50; origin xyz=0 0 0.9 rpy=0 0 0 -> xyz=0 0 0.5 rpy=0 0 0
- joint thigh_joint: limit lower=-0.523598775598 upper=3.92699081699 effort=10 velocity=5 -> lower=-0.523598775598 upper=3.92699081699 effort=100 velocity=5
